File: pcb/stm32/power_supply.kicad_sch (KiCad schematic)
At the start: 0 parts

Commit message: Power supply
Parts:
- added BT1: Battery, symbol Device:Battery
- added C4, C5, C6: 10u, symbol Device:C
- added C7: 100n, symbol Device:C
- added F1: Fuse, symbol Device:Fuse
- added L1: 4,7uH, symbol Device:L
- added Q1: ???, Package_TO_SOT_SMD:SOT-23, symbol Transistor_FET:AO3401A
- added R10, R9: 500K 1%, symbol Device:R
- added R11: 47k?, symbol Device:R
- added R12, R13: ?? 1%, symbol Device:R
- added U2: TPS61222DCK, Package_TO_SOT_SMD:Texas_R-PDSO-G6, symbol Regulator_Switching:TPS61222DCK
Connections:
- new net: F1.2, Q1.3 (D)
- new net: R12.2, R13.1, U2.2 (FB)
- new net: BT1.1 (+), F1.1
- new net: L1.2, U2.5 (L)
- new net +3.3V: C4.1, C5.1, L1.1, Q1.2 (S), R9.1, U2.1 (VIN)
- new net +5V: C6.1, C7.1, R12.1, U2.4 (VOUT)
- new net 5V_Enable: R11.1, U2.6 (EN)
- new net GND: BT1.2 (-), C4.2, C5.2, C6.2, C7.2, Q1.1 (G), R10.2, R11.2, R13.2, U2.3 (GND)
- new net VBAT_SENSE: R10.1, R9.2
Other:
- note added: "5V Supply"
- note added: "BATTERY"
- note added: "Sense"
- note added: "VDD"

Commit message: Moved PCB forwar
Parts:
- added J12: Conn_01x02_Pin, symbol Connector:Conn_01x02_Pin
- BT1: footprint (none) -> Battery:BatteryHolder_Keystone_2462_2xAA
Connections:
- net +3.3V: now also J12.1 (Pin_1); no longer C5.1, L1.1, U2.1 (VIN)
- new net: C5.1, J12.2 (Pin_2), L1.1, U2.1 (VIN)
Other:
- moved on the sheet: C5, C6, C7, L1, R11, R12, R13, U2

Commit message: Packages
Parts:
- C10: renamed from C7; footprint (none) -> Capacitor_SMD:C_0805_2012Metric
- C7: renamed from C5; footprint (none) -> Capacitor_SMD:C_0805_2012Metric
- C8: renamed from C4; footprint (none) -> Capacitor_SMD:C_0805_2012Metric
- C9: renamed from C6; footprint (none) -> Capacitor_SMD:C_0805_2012Metric
- F1: footprint (none) -> Fuse:Fuse_2920_7451Metric_Pad2.10x5.45mm_HandSolder
- J13: renamed from J12; footprint (none) -> Connector_PinHeader_2.00mm:PinHeader_1x02_P2.00mm_Vertical
- L1: footprint (none) -> Inductor_SMD:L_6.3x6.3_H3
- R11: footprint (none) -> Resistor_SMD:R_1206_3216Metric
- R12: renamed from R9; footprint (none) -> Resistor_SMD:R_1206_3216Metric
- R13: renamed from R10; footprint (none) -> Resistor_SMD:R_1206_3216Metric
- R14: renamed from R12; footprint (none) -> Resistor_SMD:R_1206_3216Metric
- R15: renamed from R13; footprint (none) -> Capacitor_SMD:C_0805_2012Metric
- renumbered U2 to U6

Commit message: VDD supply added
Changed lines of the file:
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@@
     (effects (font (size 1.27 1.27) bold) (justify left))
+  )
+  (hierarchical_label "VDD_USB" (shape input) (at 130.81 33.02 0) (fields_autoplaced)
+    (effects (font (size 1.27 1.27)) (justify left))
   )
   (symbol (lib_id "Transistor_FET:AO3401A") (at 36.83 24.13 90) (unit 1)

Commit message: PWR comment
Other:
- note added: "TODO USB to ldo to 3v3 Switch USB ldo/battery Then add jumpers to connect ldo/battery to 3v3 optional back-boost from battery to 3v3 but put usb mosfet transistor before. So we turn it off when connected to USB also add jumper to disconnect it and connect battery directly"
Changed lines of the file:
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@@
     (effects (font (size 2 2) (thickness 0.4) bold) (justify left bottom))
+  )
+  (text "TODO\n\nUSB to ldo to 3v3\nSwitch USB ldo/battery\nThen add jumpers to connect ldo/battery to 3v3\n\noptional back-boost from battery to 3v3\nbut put usb mosfet transistor before. So we turn it off when connected to USB\nalso add jumper to disconnect it and connect battery directly"
+    (at 153.67 39.37 0)
+    (effects (font (size 1.27 1.27)) (justify left bottom))
   )
   (text "5V Supply" (at 36.83 53.34 0)
