File: pcb/stm32/power_supply.kicad_sch (KiCad schematic)
At the start: 15 parts, among them J13 Conn_01x02_Pin, Q1 ???, U6 TPS61222DCK

Commit message: Progress
Other:
- note added: "TODO change footprint"
Changed lines of the file:
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@@
     (effects (font (size 2 2) (thickness 0.4) bold) (justify left bottom))
+  )
+  (text "TODO change footprint" (at 83.82 80.01 0)
+    (effects (font (size 1.27 1.27)) (justify left bottom))
   )
   (text "TODO\n\nUSB to ldo to 3v3\nSwitch USB ldo/battery\nThen add jumpers to connect ldo/battery to 3v3\n\noptional back-boost from battery to 3v3\nbut put usb mosfet transistor before. So we turn it off when connected to USB\nalso add jumper to disconnect it and connect battery directly\n\nadd another ldo after 5v to 3v3"

Commit message: Small work on pcb
Parts:
- added D2: ???, Diode_SMD:D_SOD-323, symbol Diode:SD05_SOD323
Connections:
- net GND: now also D2.1 (A1)
- net at F1.2, Q1.3 (D): now also D2.2 (A2)
Other:
- note added: "TODO: Switching USB and VCC https://electronics.stackexchange.com/questions/96059/switch-between-battery-and-usb-power-no-microcontroller-circuit"
Changed lines of the file:
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@@
   (junction (at 30.48 62.23) (diameter 0) (color 0 0 0 0)
   )
+  (junction (at 30.48 21.59) (diameter 0) (color 0 0 0 0)
+  )
   (junction (at 100.33 57.15) (diameter 0) (color 0 0 0 0)
   )
@@
   (junction (at 44.45 21.59) (diameter 0) (color 0 0 0 0)
   )
+  (junction (at 30.48 38.1) (diameter 0) (color 0 0 0 0)
+  )
   (junction (at 53.34 27.94) (diameter 0) (color 0 0 0 0)
   )
@@
     (stroke (width 0) (type default))
   )
+  (wire (pts (xy 30.48 21.59) (xy 31.75 21.59))
+    (stroke (width 0) (type default))
+  )
   (wire (pts (xy 92.71 27.94) (xy 82.55 27.94))
     (stroke (width 0) (type default))
@@
     (stroke (width 0) (type default))
   )
+  (wire (pts (xy 30.48 38.1) (xy 17.78 38.1))
+    (stroke (width 0) (type default))
+  )
   (wire (pts (xy 35.56 60.96) (xy 35.56 62.23))
     (stroke (width 0) (type default))
@@
     (stroke (width 0) (type default))
   )
-  (wire (pts (xy 29.21 21.59) (xy 31.75 21.59))
+  (wire (pts (xy 29.21 21.59) (xy 30.48 21.59))
     (stroke (width 0) (type default))
   )
@@
     (stroke (width 0) (type default))
   )
+  (wire (pts (xy 30.48 21.59) (xy 30.48 27.94))
+    (stroke (width 0) (type default))
+  )
   (wire (pts (xy 17.78 21.59) (xy 21.59 21.59))
     (stroke (width 0) (type default))
@@
     (stroke (width 0) (type default))
   )
+  (wire (pts (xy 30.48 35.56) (xy 30.48 38.1))
+    (stroke (width 0) (type default))
+  )
   (wire (pts (xy 53.34 27.94) (xy 55.88 27.94))
     (stroke (width 0) (type default))
@@
     (stroke (width 0) (type default))
   )
-  (wire (pts (xy 36.83 38.1) (xy 17.78 38.1))
+  (wire (pts (xy 36.83 38.1) (xy 30.48 38.1))
     (stroke (width 0) (type default))
   )
@@
   )
   (text "TODO change footprint" (at 83.82 80.01 0)
+    (effects (font (size 1.27 1.27)) (justify left bottom))
+  )
+  (text "TODO: Switching USB and VCC \nhttps://electronics.stackexchange.com/questions/96059/switch-between-battery-and-usb-power-no-microcontroller-circuit"
+    (at 130.81 58.42 0)
     (effects (font (size 1.27 1.27)) (justify left bottom))
   )
@@
         )
       )
+    )
+  )
+  (symbol (lib_id "Diode:SD05_SOD323") (at 30.48 31.75 90) (unit 1)
+    (in_bom yes) (on_board yes) (dnp no) (fields_autoplaced)
+    (property "Reference" "D2" (at 33.02 31.115 90)
+      (effects (font (size 1.27 1.27)) (justify right))
+    )
+    (property "Value" "???" (at 33.02 33.655 90)
+      (effects (font (size 1.27 1.27)) (justify right))
+    )
+    (property "Footprint" "Diode_SMD:D_SOD-323" (at 35.56 31.75 0)
+      (effects (font (size 1.27 1.27)) hide)
+    )
+    (property "Datasheet" "https://www.littelfuse.com/~/media/electronics/datasheets/tvs_diode_arrays/littelfuse_tvs_diode_array_sd_c_datasheet.pdf.pdf" (at 30.48 31.75 0)
+      (effects (font (size 1.27 1.27)) hide)
+    )
+    (pin "1")
+    (pin "2")
+    (instances
+      (project "stm32"
+        (path "/cc56704c-71b4-401e-bec6-203f83946289/8878edf1-eecf-4d8b-8425-07bf183b31b3"
+          (reference "D2") (unit 1)
+        )
+      )

Commit message: WIP pcb
Parts:
- added Q2: DMG3415, Package_TO_SOT_SMD:SOT-23, symbol Transistor_FET:DMG2301L
- added U10: TPL5110, Package_TO_SOT_SMD:SOT-23-6, symbol Timer:TPL5110
Other:
- note added: "See: https://cdn-learn.adafruit.com/assets/assets/000/039/783/original/adafruit_products_schem.png?1488404279"
Changed lines of the file:
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@@
     (effects (font (size 2 2) (thickness 0.4) bold) (justify left bottom))
+  )
+  (text "See: https://cdn-learn.adafruit.com/assets/assets/000/039/783/original/adafruit_products_schem.png?1488404279"
+    (at 143.51 109.22 0)
+    (effects (font (size 1.27 1.27)) (justify left bottom))
   )
   (text "TODO change footprint" (at 83.82 80.01 0)
@@
         (path "/cc56704c-71b4-401e-bec6-203f83946289/8878edf1-eecf-4d8b-8425-07bf183b31b3"
           (reference "F1") (unit 1)
+        )
+      )
+    )
+  )
+  (symbol (lib_id "Transistor_FET:DMG2301L") (at 194.31 120.65 270) (mirror x) (unit 1)
+    (in_bom yes) (on_board yes) (dnp no)
+    (property "Reference" "Q2" (at 194.31 111.76 90)
+      (effects (font (size 1.27 1.27)))
+    )
+    (property "Value" "DMG3415" (at 194.31 114.3 90)
+      (effects (font (size 1.27 1.27)))
+    )
+    (property "Footprint" "Package_TO_SOT_SMD:SOT-23" (at 192.405 115.57 0)
+      (effects (font (size 1.27 1.27) italic) (justify left) hide)
+    )
+    (property "Datasheet" "https://www.diodes.com/assets/Datasheets/DMG2301L.pdf" (at 194.31 120.65 0)
+      (effects (font (size 1.27 1.27)) (justify left) hide)
+    )
+    (pin "1")
+    (pin "2")
+    (pin "3")
+    (instances
+      (project "stm32"
+        (path "/cc56704c-71b4-401e-bec6-203f83946289"
+          (reference "Q2") (unit 1)
+        )
+        (path "/cc56704c-71b4-401e-bec6-203f83946289/8878edf1-eecf-4d8b-8425-07bf183b31b3"
+          (reference "Q2") (unit 1)
         )
       )
@@
         )
       )
+    )
+  )
+  (symbol (lib_id "Timer:TPL5110") (at 168.91 132.08 0) (unit 1)
+    (in_bom yes) (on_board yes) (dnp no) (fields_autoplaced)
+    (property "Reference" "U10" (at 170.8659 120.65 0)
+      (effects (font (size 1.27 1.27)) (justify left))
+    )
+    (property "Value" "TPL5110" (at 170.8659 123.19 0)
+      (effects (font (size 1.27 1.27)) (justify left))
+    )
+    (property "Footprint" "Package_TO_SOT_SMD:SOT-23-6" (at 168.91 132.08 0)
+      (effects (font (size 1.27 1.27)) hide)
+    )
+    (property "Datasheet" "http://www.ti.com/lit/ds/symlink/tpl5110.pdf" (at 163.83 142.24 0)
+      (effects (font (size 1.27 1.27)) hide)
+    )
+    (pin "1")
+    (pin "2")
+    (pin "3")
+    (pin "4")
+    (pin "5")
+    (pin "6")
+    (instances
+      (project "stm32"
+        (path "/cc56704c-71b4-401e-bec6-203f83946289"
+          (reference "U10") (unit 1)
+        )
+        (path "/cc56704c-71b4-401e-bec6-203f83946289/8878edf1-eecf-4d8b-8425-07bf183b31b3"
+          (reference "U10") (unit 1)
+        )
+      )

Commit message: update
Parts:
- removed Q2: DMG3415, Package_TO_SOT_SMD:SOT-23, symbol Transistor_FET:DMG2301L
- removed U10: TPL5110, Package_TO_SOT_SMD:SOT-23-6, symbol Timer:TPL5110
Other:
- note added: "See: https://cdn-learn.adafruit.com/assets/assets/000/039/783/original/adafruit_products_schem.png?1488404279 TPL5110 + mosfet DMG3415"
- note removed: "See: https://cdn-learn.adafruit.com/assets/assets/000/039/783/original/adafruit_products_schem.png?1488404279"
Changed lines of the file:
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@@
     (effects (font (size 2 2) (thickness 0.4) bold) (justify left bottom))
   )
-  (text "See: https://cdn-learn.adafruit.com/assets/assets/000/039/783/original/adafruit_products_schem.png?1488404279"
+  (text "See: https://cdn-learn.adafruit.com/assets/assets/000/039/783/original/adafruit_products_schem.png?1488404279\nTPL5110 + mosfet DMG3415\n"
     (at 143.51 109.22 0)
     (effects (font (size 1.27 1.27)) (justify left bottom))
@@
         (path "/cc56704c-71b4-401e-bec6-203f83946289/8878edf1-eecf-4d8b-8425-07bf183b31b3"
           (reference "F1") (unit 1)
-        )
-      )
-    )
-  )
-  (symbol (lib_id "Transistor_FET:DMG2301L") (at 194.31 120.65 270) (mirror x) (unit 1)
-    (in_bom yes) (on_board yes) (dnp no)
-    (property "Reference" "Q2" (at 194.31 111.76 90)
-      (effects (font (size 1.27 1.27)))
-    )
-    (property "Value" "DMG3415" (at 194.31 114.3 90)
-      (effects (font (size 1.27 1.27)))
-    )
-    (property "Footprint" "Package_TO_SOT_SMD:SOT-23" (at 192.405 115.57 0)
-      (effects (font (size 1.27 1.27) italic) (justify left) hide)
-    )
-    (property "Datasheet" "https://www.diodes.com/assets/Datasheets/DMG2301L.pdf" (at 194.31 120.65 0)
-      (effects (font (size 1.27 1.27)) (justify left) hide)
-    )
-    (pin "1")
-    (pin "2")
-    (pin "3")
-    (instances
-      (project "stm32"
-        (path "/cc56704c-71b4-401e-bec6-203f83946289"
-          (reference "Q2") (unit 1)
-        )
-        (path "/cc56704c-71b4-401e-bec6-203f83946289/8878edf1-eecf-4d8b-8425-07bf183b31b3"
-          (reference "Q2") (unit 1)
         )
       )
@@
         )
       )
-    )
-  )
-  (symbol (lib_id "Timer:TPL5110") (at 168.91 132.08 0) (unit 1)
-    (in_bom yes) (on_board yes) (dnp no) (fields_autoplaced)
-    (property "Reference" "U10" (at 170.8659 120.65 0)
-      (effects (font (size 1.27 1.27)) (justify left))
-    )
-    (property "Value" "TPL5110" (at 170.8659 123.19 0)
-      (effects (font (size 1.27 1.27)) (justify left))
-    )
-    (property "Footprint" "Package_TO_SOT_SMD:SOT-23-6" (at 168.91 132.08 0)
-      (effects (font (size 1.27 1.27)) hide)
-    )
-    (property "Datasheet" "http://www.ti.com/lit/ds/symlink/tpl5110.pdf" (at 163.83 142.24 0)
-      (effects (font (size 1.27 1.27)) hide)
-    )
-    (pin "1")
-    (pin "2")
-    (pin "3")
-    (pin "4")
-    (pin "5")
-    (pin "6")
-    (instances
-      (project "stm32"
-        (path "/cc56704c-71b4-401e-bec6-203f83946289"
-          (reference "U10") (unit 1)
-        )
-        (path "/cc56704c-71b4-401e-bec6-203f83946289/8878edf1-eecf-4d8b-8425-07bf183b31b3"
-          (reference "U10") (unit 1)
-        )
-      )

Commit message: update schema
Parts:
- added C11: 10u, Capacitor_SMD:C_0805_2012Metric, symbol Device:C
- added C12: 100n, Capacitor_SMD:C_0805_2012Metric, symbol Device:C
- added D4: 1N5819, Diode_THT:D_DO-41_SOD81_P10.16mm_Horizontal, symbol Diode:1N5819
- added Q2: SI4427, Package_TO_SOT_SMD:SOT-23, symbol Transistor_FET:AO3401A
- added R16: 470k, Resistor_SMD:R_1206_3216Metric, symbol Device:R
- added U10: LTC4412xS6, Package_TO_SOT_SMD:TSOT-23-6, symbol Power_Management:LTC4412xS6
- added U11: AMS1117-3.3, Package_TO_SOT_SMD:SOT-223-3_TabPin2, symbol Regulator_Linear:AMS1117-3.3
- Q1: value ??? -> SI4427
Connections:
- net +3.3V: now also C11.1, C12.1, D4.1 (K), Q2.2 (S), R16.1, U10.6 (SENSE); no longer C8.1, Q1.2 (S), R12.1
- net GND: now also C11.2, C12.2, U10.2 (GND), U10.3 (CTL), U11.1 (GND)
- net VDD_USB: now also U11.3 (VI)
- new net: Q2.1 (G), U10.5 (GATE)
- new net: D4.2 (A), U11.2 (VO)
- new net: R16.2, U10.4 (STAT)
- new net +BATT: C8.1, Q1.2 (S), Q2.3 (D), R12.1, U10.1 (VIN)
Other:
- note added: "CHECK DONE"
- note added: "TODO: Switching USB and VCC https://electronics.stackexchange.com/questions/96059/switch-between-battery-and-usb-power-no-microcontroller-circuit https://electronics.stackexchange.com/questions/130932/switching-between-battery-and-usb-using-diode-or-logic"
- note added: "USB / Batt switch"
- note removed: "TODO: Switching USB and VCC https://electronics.stackexchange.com/questions/96059/switch-between-battery-and-usb-power-no-microcontroller-circuit"
- note removed: "VDD"
