File: pcb/stm32/sensors_i2c.kicad_sch (KiCad schematic)
At the start: 0 parts

Commit message: Packages
Parts:
- added U7: BME280, Package_LGA:Bosch_LGA-8_2.5x2.5mm_P0.65mm_ClockwisePinNumbering, symbol Sensor:BME280
Changed lines of the file:
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@@
     (effects (font (size 1.27 1.27) bold) (justify left))
   )
+  (symbol (lib_id "Sensor:BME280") (at 67.31 54.61 0) (unit 1)
+    (in_bom yes) (on_board yes) (dnp no) (fields_autoplaced)
+    (property "Reference" "U7" (at 55.88 53.975 0)
+      (effects (font (size 1.27 1.27)) (justify right))
+    )
+    (property "Value" "BME280" (at 55.88 56.515 0)
+      (effects (font (size 1.27 1.27)) (justify right))
+    )
+    (property "Footprint" "Package_LGA:Bosch_LGA-8_2.5x2.5mm_P0.65mm_ClockwisePinNumbering" (at 105.41 66.04 0)
+      (effects (font (size 1.27 1.27)) hide)
+    )
+    (property "Datasheet" "https://www.bosch-sensortec.com/media/boschsensortec/downloads/datasheets/bst-bme280-ds002.pdf" (at 67.31 59.69 0)
+      (effects (font (size 1.27 1.27)) hide)
+    )
+    (pin "1")
+    (pin "2")
+    (pin "3")
+    (pin "4")
+    (pin "5")
+    (pin "6")
+    (pin "7")
+    (pin "8")
+    (instances
+      (project "stm32"
+        (path "/cc56704c-71b4-401e-bec6-203f83946289/2f9a377a-ab8f-4f3f-978d-a700fa170109"
+          (reference "U7") (unit 1)
+        )
+      )
+    )
+  )
 )

Commit message: Added todos
Other:
- note added: "TODO: light sensor from laskakit"
Changed lines of the file:
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@@
 (kicad_sch (version 20230121) (generator eeschema)
   (paper "A4")
+  (text "TODO: light sensor from laskakit" (at 57.15 33.02 0)
+    (effects (font (face "KiCad Font") (size 3 3)) (justify left bottom))
+  )
   (hierarchical_label "VDD" (shape input) (at 90.17 91.44 0) (fields_autoplaced)
     (effects (font (size 1.27 1.27) bold) (justify left))
