File: pcb/stm32/stm32_core.kicad_sch (KiCad schematic)
At the start: 21 parts, among them J1 Conn_01x04_Pin, J2 Conn_01x06_Pin, J3 Conn_02x05_Top_Bottom, J4 Conn_01x02_Pin, J5 Conn_02x05_Top_Bottom, J6 Conn_01x02_Pin, SW1 SW_Push, SW2 SW_Push, SW3 SW_Push, U1 STM32G070KBT6

Commit message: Moved PCB forwar
Parts:
- added J11: Conn_01x06_Pin, symbol Connector:Conn_01x06_Pin
Connections:
- net +3.3V: now also J11.1 (Pin_1)
- net GND: now also J11.6 (Pin_6)
- net SPI_MISO: now also J11.3 (Pin_3)
- net SPI_MOSI: now also J11.4 (Pin_4)
- net SPI_SCK: now also J11.2 (Pin_2)
- net SPI_SS2: now also J11.5 (Pin_5)
- net Battery_ADC renamed BAT_SENSE
Other:
- note added: "SPI"

Commit message: Packages
Parts:
- C4: renamed from C1; footprint (none) -> Capacitor_SMD:C_0201_0603Metric
- C5: renamed from C3; footprint (none) -> Capacitor_SMD:C_0201_0603Metric
- C6: renamed from C2; footprint (none) -> Capacitor_SMD:C_0805_2012Metric
- J2: renamed from J4; footprint (none) -> Connector_PinHeader_2.00mm:PinHeader_1x02_P2.00mm_Vertical
- J3: renamed from J5; footprint (none) -> Connector_PinHeader_2.00mm:PinHeader_2x05_P2.00mm_Vertical
- J4: renamed from J11; footprint (none) -> Connector_PinHeader_2.00mm:PinHeader_1x06_P2.00mm_Vertical
- J5: renamed from J3; footprint (none) -> Connector_PinHeader_2.00mm:PinHeader_2x05_P2.00mm_Vertical
- J6: renamed from J2; footprint (none) -> Connector_PinHeader_2.00mm:PinHeader_1x06_P2.00mm_Vertical
- J7: renamed from J1; footprint (none) -> Connector_PinHeader_2.00mm:PinHeader_1x04_P2.00mm_Vertical
- J8: renamed from J6; footprint (none) -> Connector_PinHeader_2.00mm:PinHeader_1x03_P2.00mm_Vertical
- R10: renamed from R8; footprint (none) -> Resistor_SMD:R_1206_3216Metric
- R3: renamed from R1; footprint (none) -> Resistor_SMD:R_1206_3216Metric
- R4: renamed from R2; footprint (none) -> Resistor_SMD:R_1206_3216Metric
- R5: footprint (none) -> Resistor_SMD:R_1206_3216Metric
- R6: renamed from R3; footprint (none) -> Resistor_SMD:R_1206_3216Metric
- R7: renamed from R4; footprint (none) -> Resistor_SMD:R_1206_3216Metric
- R8: renamed from R6; footprint (none) -> Resistor_SMD:R_1206_3216Metric
- R9: renamed from R7; footprint (none) -> Resistor_SMD:R_1206_3216Metric
- SW1, SW2, SW3: footprint (none) -> Button_Switch_SMD:SW_SPST_PTS810
- U4: renamed from U1; footprint LQFP-32 -> Package_QFP:LQFP-32_7x7mm_P0.8mm

Commit message: Added todos
Other:
- note added: "TODO: Add spare pins to a header for dev board"
Changed lines of the file:
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@@
     (fill (type none))
+  )
+  (text "TODO: Add spare pins to a header for dev board\n" (at 128.27 144.78 0)
+    (effects (font (size 3 3)) (justify left bottom))
   )
   (text "I2C" (at 15.24 26.67 0)

Commit message: update schema
Parts:
- added J17: Conn_01x11, symbol Connector_Generic:Conn_01x11
- SW3: value SW_Push -> Reset
Connections:
- net +3.3V: now also J17.1 (Pin_1)
- net GND: now also J17.11 (Pin_11)
- net PA3: now reaches U4.10 (PA3)
- net PA3: now also J17.3 (Pin_3)
- net PC6: now reaches U4.20 (PC6)
- net PC6: now also J17.10 (Pin_10)
- net PA15: now reaches U4.26 (PA15)
- net PA15: now also J17.4 (Pin_4)
- net PB3: now reaches U4.27 (PB3)
- net PB3: now also J17.5 (Pin_5)
- net PB4: now reaches U4.28 (PB4)
- net PB4: now also J17.6 (Pin_6)
- net PB5: now reaches U4.29 (PB5)
- net PB5: now also J17.7 (Pin_7)
- net PB7: now reaches U4.31 (PB7)
- net PB7: now also J17.8 (Pin_8)
- net PB8: now reaches U4.32 (PB8)
- net PB8: now also J17.9 (Pin_9)
- net PA2: now reaches U4.9 (PA2)
- net PA2: now also J17.2 (Pin_2)
- no-connect marks 13 -> 4
Other:
- note added: "CHECK DONE"
- note added: "Not used pins"
- note removed: "TODO: Add spare pins to a header for dev board"
