File: pcb/stm32/sensors_onewire.kicad_sch (KiCad schematic)
At the start: 2 parts, among them J7 4P4C, J8 4P4C

Commit message: Moved PCB forwar
Changed lines of the file:
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@@
 (kicad_sch (version 20230121) (generator eeschema)
   (paper "A4")
+  (hierarchical_label "VDD" (shape input) (at 121.92 81.28 0) (fields_autoplaced)
+    (effects (font (size 1.27 1.27) bold) (justify left))
+  )
+  (hierarchical_label "GND" (shape input) (at 121.92 85.09 0) (fields_autoplaced)
+    (effects (font (size 1.27 1.27) bold) (justify left))
+  )
+  (hierarchical_label "OneWire" (shape bidirectional) (at 121.92 77.47 0) (fields_autoplaced)
+    (effects (font (size 1.27 1.27) bold) (justify left))
+  )
   (symbol (lib_id "Connector:4P4C") (at 59.69 68.58 0) (unit 1)
     (in_bom yes) (on_board yes) (dnp no) (fields_autoplaced)

Commit message: Packages
Parts:
- added J11, J12: 4P4C, Connector_RJ:RJ14_Connfly_DS1133-S4_Horizontal, symbol Connector:4P4C
- added U5: DS18B20, Package_TO_SOT_THT:TO-92_Inline, symbol Sensor_Temperature:DS18B20
- J10: renamed from J8; footprint (none) -> Connector_RJ:RJ14_Connfly_DS1133-S4_Horizontal
- J9: renamed from J7; footprint (none) -> Connector_RJ:RJ14_Connfly_DS1133-S4_Horizontal
Changed lines of the file:
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@@
     (effects (font (size 1.27 1.27) bold) (justify left))
+  )
+  (symbol (lib_id "Sensor_Temperature:DS18B20") (at 111.76 41.91 0) (unit 1)
+    (in_bom yes) (on_board yes) (dnp no) (fields_autoplaced)
+    (property "Reference" "U5" (at 105.41 41.275 0)
+      (effects (font (size 1.27 1.27)) (justify right))
+    )
+    (property "Value" "DS18B20" (at 105.41 43.815 0)
+      (effects (font (size 1.27 1.27)) (justify right))
+    )
+    (property "Footprint" "Package_TO_SOT_THT:TO-92_Inline" (at 86.36 48.26 0)
+      (effects (font (size 1.27 1.27)) hide)
+    )
+    (property "Datasheet" "http://datasheets.maximintegrated.com/en/ds/DS18B20.pdf" (at 107.95 35.56 0)
+      (effects (font (size 1.27 1.27)) hide)
+    )
+    (pin "1")
+    (pin "2")
+    (pin "3")
+    (instances
+      (project "stm32"
+        (path "/cc56704c-71b4-401e-bec6-203f83946289/10666af3-dfc7-46de-8942-14bdd4d81ac1"
+          (reference "U5") (unit 1)
+        )
+      )
+    )
+  )
+  (symbol (lib_id "Connector:4P4C") (at 59.69 87.63 0) (unit 1)
+    (in_bom yes) (on_board yes) (dnp no) (fields_autoplaced)
+    (property "Reference" "J11" (at 59.69 76.2 0)
+      (effects (font (size 1.27 1.27)))
+    )
+    (property "Value" "4P4C" (at 59.69 78.74 0)
+      (effects (font (size 1.27 1.27)))
+    )
+    (property "Footprint" "Connector_RJ:RJ14_Connfly_DS1133-S4_Horizontal" (at 59.69 86.36 90)
+      (effects (font (size 1.27 1.27)) hide)
+    )
+    (property "Datasheet" "~" (at 59.69 86.36 90)
+      (effects (font (size 1.27 1.27)) hide)
+    )
+    (pin "1")
+    (pin "2")
+    (pin "3")
+    (pin "4")
+    (instances
+      (project "stm32"
+        (path "/cc56704c-71b4-401e-bec6-203f83946289/10666af3-dfc7-46de-8942-14bdd4d81ac1"
+          (reference "J11") (unit 1)
+        )
+      )
+    )
   )
   (symbol (lib_id "Connector:4P4C") (at 59.69 68.58 0) (unit 1)
     (in_bom yes) (on_board yes) (dnp no) (fields_autoplaced)
-    (property "Reference" "J8" (at 59.69 57.15 0)
+    (property "Reference" "J10" (at 59.69 57.15 0)
       (effects (font (size 1.27 1.27)))
     )
@@
       (effects (font (size 1.27 1.27)))
     )
-    (property "Footprint" "" (at 59.69 67.31 90)
+    (property "Footprint" "Connector_RJ:RJ14_Connfly_DS1133-S4_Horizontal" (at 59.69 67.31 90)
       (effects (font (size 1.27 1.27)) hide)
     )
@@
       (project "stm32"
         (path "/cc56704c-71b4-401e-bec6-203f83946289/10666af3-dfc7-46de-8942-14bdd4d81ac1"
-          (reference "J8") (unit 1)
+          (reference "J10") (unit 1)
+        )
+      )
+    )
+  )
+  (symbol (lib_id "Connector:4P4C") (at 59.69 106.68 0) (unit 1)
+    (in_bom yes) (on_board yes) (dnp no) (fields_autoplaced)
+    (property "Reference" "J12" (at 59.69 95.25 0)
+      (effects (font (size 1.27 1.27)))
+    )
+    (property "Value" "4P4C" (at 59.69 97.79 0)
+      (effects (font (size 1.27 1.27)))
+    )
+    (property "Footprint" "Connector_RJ:RJ14_Connfly_DS1133-S4_Horizontal" (at 59.69 105.41 90)
+      (effects (font (size 1.27 1.27)) hide)
+    )
+    (property "Datasheet" "~" (at 59.69 105.41 90)
+      (effects (font (size 1.27 1.27)) hide)
+    )
+    (pin "1")
+    (pin "2")
+    (pin "3")
+    (pin "4")
+    (instances
+      (project "stm32"
+        (path "/cc56704c-71b4-401e-bec6-203f83946289/10666af3-dfc7-46de-8942-14bdd4d81ac1"
+          (reference "J12") (unit 1)
         )
       )
@@
   (symbol (lib_id "Connector:4P4C") (at 59.69 49.53 0) (unit 1)
     (in_bom yes) (on_board yes) (dnp no) (fields_autoplaced)
-    (property "Reference" "J7" (at 59.69 38.1 0)
+    (property "Reference" "J9" (at 59.69 38.1 0)
       (effects (font (size 1.27 1.27)))
     )
@@
       (effects (font (size 1.27 1.27)))
     )
-    (property "Footprint" "" (at 59.69 48.26 90)
+    (property "Footprint" "Connector_RJ:RJ14_Connfly_DS1133-S4_Horizontal" (at 59.69 48.26 90)
       (effects (font (size 1.27 1.27)) hide)
     )
@@
       (project "stm32"
         (path "/cc56704c-71b4-401e-bec6-203f83946289/10666af3-dfc7-46de-8942-14bdd4d81ac1"
-          (reference "J7") (unit 1)
+          (reference "J9") (unit 1)
         )
       )

Commit message: Small updates on pcb
Parts:
- removed J10, J11, J12, J9: 4P4C, Connector_RJ:RJ14_Connfly_DS1133-S4_Horizontal, symbol Connector:4P4C
Other:
- note added: "Check out https://www.lcsc.com/product-detail/Ethernet-Connectors-Modular-Connectors-span-style-background-color-ff0-RJ45-span-RJ11_CONNFLY-Elec-DS1129-02-S80BP_C77852.html and wiring https://rpishop.cz/1-wire/5689-1wire-teplotni-senzor-15-m.html"
Changed lines of the file:
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@@
 (kicad_sch (version 20230121) (generator eeschema)
   (paper "A4")
+  (text "Check out\nhttps://www.lcsc.com/product-detail/Ethernet-Connectors-Modular-Connectors-span-style-background-color-ff0-RJ45-span-RJ11_CONNFLY-Elec-DS1129-02-S80BP_C77852.html\n\nand wiring\nhttps://rpishop.cz/1-wire/5689-1wire-teplotni-senzor-15-m.html"
+    (at 36.83 129.54 0)
+    (effects (font (size 1.27 1.27)) (justify left bottom))
+  )
   (hierarchical_label "VDD" (shape input) (at 121.92 81.28 0) (fields_autoplaced)
     (effects (font (size 1.27 1.27) bold) (justify left))
@@
         )
       )
-    )
-  )
-  (symbol (lib_id "Connector:4P4C") (at 59.69 87.63 0) (unit 1)
-    (in_bom yes) (on_board yes) (dnp no) (fields_autoplaced)
-    (property "Reference" "J11" (at 59.69 76.2 0)
-      (effects (font (size 1.27 1.27)))
-    )
-    (property "Value" "4P4C" (at 59.69 78.74 0)
-      (effects (font (size 1.27 1.27)))
-    )
-    (property "Footprint" "Connector_RJ:RJ14_Connfly_DS1133-S4_Horizontal" (at 59.69 86.36 90)
-      (effects (font (size 1.27 1.27)) hide)
-    )
-    (property "Datasheet" "~" (at 59.69 86.36 90)
-      (effects (font (size 1.27 1.27)) hide)
-    )
-    (pin "1")
-    (pin "2")
-    (pin "3")
-    (pin "4")
-    (instances
-      (project "stm32"
-        (path "/cc56704c-71b4-401e-bec6-203f83946289/10666af3-dfc7-46de-8942-14bdd4d81ac1"
-          (reference "J11") (unit 1)
-        )
-      )
-    )
-  )
-  (symbol (lib_id "Connector:4P4C") (at 59.69 68.58 0) (unit 1)
-    (in_bom yes) (on_board yes) (dnp no) (fields_autoplaced)
-    (property "Reference" "J10" (at 59.69 57.15 0)
-      (effects (font (size 1.27 1.27)))
-    )
-    (property "Value" "4P4C" (at 59.69 59.69 0)
-      (effects (font (size 1.27 1.27)))
-    )
-    (property "Footprint" "Connector_RJ:RJ14_Connfly_DS1133-S4_Horizontal" (at 59.69 67.31 90)
-      (effects (font (size 1.27 1.27)) hide)
-    )
-    (property "Datasheet" "~" (at 59.69 67.31 90)
-      (effects (font (size 1.27 1.27)) hide)
-    )
-    (pin "1")
-    (pin "2")
-    (pin "3")
-    (pin "4")
-    (instances
-      (project "stm32"
-        (path "/cc56704c-71b4-401e-bec6-203f83946289/10666af3-dfc7-46de-8942-14bdd4d81ac1"
-          (reference "J10") (unit 1)
-        )
-      )
-    )
-  )
-  (symbol (lib_id "Connector:4P4C") (at 59.69 106.68 0) (unit 1)
-    (in_bom yes) (on_board yes) (dnp no) (fields_autoplaced)
-    (property "Reference" "J12" (at 59.69 95.25 0)
-      (effects (font (size 1.27 1.27)))
-    )
-    (property "Value" "4P4C" (at 59.69 97.79 0)
-      (effects (font (size 1.27 1.27)))
-    )
-    (property "Footprint" "Connector_RJ:RJ14_Connfly_DS1133-S4_Horizontal" (at 59.69 105.41 90)
-      (effects (font (size 1.27 1.27)) hide)
-    )
-    (property "Datasheet" "~" (at 59.69 105.41 90)
-      (effects (font (size 1.27 1.27)) hide)
-    )
-    (pin "1")
-    (pin "2")
-    (pin "3")
-    (pin "4")
-    (instances
-      (project "stm32"
-        (path "/cc56704c-71b4-401e-bec6-203f83946289/10666af3-dfc7-46de-8942-14bdd4d81ac1"
-          (reference "J12") (unit 1)
-        )
-      )
-    )
-  )
-  (symbol (lib_id "Connector:4P4C") (at 59.69 49.53 0) (unit 1)
-    (in_bom yes) (on_board yes) (dnp no) (fields_autoplaced)
-    (property "Reference" "J9" (at 59.69 38.1 0)
-      (effects (font (size 1.27 1.27)))
-    )
-    (property "Value" "4P4C" (at 59.69 40.64 0)
-      (effects (font (size 1.27 1.27)))
-    )
-    (property "Footprint" "Connector_RJ:RJ14_Connfly_DS1133-S4_Horizontal" (at 59.69 48.26 90)
-      (effects (font (size 1.27 1.27)) hide)
-    )
-    (property "Datasheet" "~" (at 59.69 48.26 90)
-      (effects (font (size 1.27 1.27)) hide)
-    )
-    (pin "1")
-    (pin "2")
-    (pin "3")
-    (pin "4")
-    (instances
-      (project "stm32"
-        (path "/cc56704c-71b4-401e-bec6-203f83946289/10666af3-dfc7-46de-8942-14bdd4d81ac1"
-          (reference "J9") (unit 1)
-        )
-      )
