File: pcb/stm32/wireless.kicad_sch (KiCad schematic)
At the start: 2 parts, among them J7 4P4C

Commit message: Moved PCB forwar
Changed lines of the file:
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@@
 (kicad_sch (version 20230121) (generator eeschema)
   (paper "A4")
+  (hierarchical_label "RF_RX" (shape output) (at 140.97 77.47 0) (fields_autoplaced)
+    (effects (font (size 1.27 1.27) bold) (justify left))
+  )
+  (hierarchical_label "RF_TX" (shape input) (at 140.97 73.66 0) (fields_autoplaced)
+    (effects (font (size 1.27 1.27) bold) (justify left))
+  )
+  (hierarchical_label "VDD" (shape input) (at 142.24 87.63 0) (fields_autoplaced)
+    (effects (font (size 1.27 1.27) bold) (justify left))
+  )
+  (hierarchical_label "GND" (shape input) (at 142.24 91.44 0) (fields_autoplaced)
+    (effects (font (size 1.27 1.27) bold) (justify left))
+  )
   (symbol (lib_id "Connector:4P4C") (at 72.39 72.39 0) (unit 1)
     (in_bom yes) (on_board yes) (dnp no) (fields_autoplaced)

Commit message: Packages
Parts:
- J7: footprint (none) -> Connector_RJ:RJ14_Connfly_DS1133-S4_Horizontal
Changed lines of the file:
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@@
       (effects (font (size 1.27 1.27)))
     )
-    (property "Footprint" "" (at 72.39 71.12 90)
+    (property "Footprint" "Connector_RJ:RJ14_Connfly_DS1133-S4_Horizontal" (at 72.39 71.12 90)
       (effects (font (size 1.27 1.27)) hide)
     )
@@
         )
         (path "/cc56704c-71b4-401e-bec6-203f83946289/373d422b-50db-40b1-b72f-ec977be46bcc"
-          (reference "J9") (unit 1)
+          (reference "J14") (unit 1)
         )
       )
@@
       (effects (font (size 1.27 1.27)))
     )
-    (property "Footprint" "" (at 72.39 90.17 90)
+    (property "Footprint" "Connector_RJ:RJ14_Connfly_DS1133-S4_Horizontal" (at 72.39 90.17 90)
       (effects (font (size 1.27 1.27)) hide)
     )
@@
         )
         (path "/cc56704c-71b4-401e-bec6-203f83946289/373d422b-50db-40b1-b72f-ec977be46bcc"
-          (reference "J10") (unit 1)
+          (reference "J15") (unit 1)
         )
       )

Commit message: Added todos
Other:
- note added: "Interface before wireless to be able to connect by wire"
Changed lines of the file:
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@@
 (kicad_sch (version 20230121) (generator eeschema)
   (paper "A4")
+  (text "Interface before wireless\nto be able to connect by wire\n"
+    (at 63.5 58.42 0)
+    (effects (font (size 1.27 1.27)) (justify left bottom))
+  )
   (hierarchical_label "RF_RX" (shape output) (at 140.97 77.47 0) (fields_autoplaced)
     (effects (font (size 1.27 1.27) bold) (justify left))

Commit message: Small updates on pcb
Parts:
- removed J7 (x2): 4P4C, Connector_RJ:RJ14_Connfly_DS1133-S4_Horizontal, symbol Connector:4P4C
Other:
- note added: "Checkout https://www.lcsc.com/product-detail/Ethernet-Connectors-Modular-Connectors-span-style-background-color-ff0-RJ45-span-RJ11_Ckmtw-Shenzhen-Cankemeng-R-RJ45R08P-2006_C386761.html"
Changed lines of the file:
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@@
 (kicad_sch (version 20230121) (generator eeschema)
   (paper "A4")
+  (text "Checkout\n\nhttps://www.lcsc.com/product-detail/Ethernet-Connectors-Modular-Connectors-span-style-background-color-ff0-RJ45-span-RJ11_Ckmtw-Shenzhen-Cankemeng-R-RJ45R08P-2006_C386761.html\n"
+    (at 43.18 105.41 0)
+    (effects (font (size 1.27 1.27)) (justify left bottom))
+  )
   (text "Interface before wireless\nto be able to connect by wire\n"
     (at 63.5 58.42 0)
@@
     (effects (font (size 1.27 1.27) bold) (justify left))
   )
-  (symbol (lib_id "Connector:4P4C") (at 72.39 72.39 0) (unit 1)
-    (in_bom yes) (on_board yes) (dnp no) (fields_autoplaced)
-    (property "Reference" "J7" (at 72.39 60.96 0)
-      (effects (font (size 1.27 1.27)))
-    )
-    (property "Value" "4P4C" (at 72.39 63.5 0)
-      (effects (font (size 1.27 1.27)))
-    )
-    (property "Footprint" "Connector_RJ:RJ14_Connfly_DS1133-S4_Horizontal" (at 72.39 71.12 90)
-      (effects (font (size 1.27 1.27)) hide)
-    )
-    (property "Datasheet" "~" (at 72.39 71.12 90)
-      (effects (font (size 1.27 1.27)) hide)
-    )
-    (pin "1")
-    (pin "2")
-    (pin "3")
-    (pin "4")
-    (instances
-      (project "stm32"
-        (path "/cc56704c-71b4-401e-bec6-203f83946289/10666af3-dfc7-46de-8942-14bdd4d81ac1"
-          (reference "J7") (unit 1)
-        )
-        (path "/cc56704c-71b4-401e-bec6-203f83946289/373d422b-50db-40b1-b72f-ec977be46bcc"
-          (reference "J14") (unit 1)
-        )
-      )
-    )
-  )
-  (symbol (lib_id "Connector:4P4C") (at 72.39 91.44 0) (unit 1)
-    (in_bom yes) (on_board yes) (dnp no) (fields_autoplaced)
-    (property "Reference" "J7" (at 72.39 80.01 0)
-      (effects (font (size 1.27 1.27)))
-    )
-    (property "Value" "4P4C" (at 72.39 82.55 0)
-      (effects (font (size 1.27 1.27)))
-    )
-    (property "Footprint" "Connector_RJ:RJ14_Connfly_DS1133-S4_Horizontal" (at 72.39 90.17 90)
-      (effects (font (size 1.27 1.27)) hide)
-    )
-    (property "Datasheet" "~" (at 72.39 90.17 90)
-      (effects (font (size 1.27 1.27)) hide)
-    )
-    (pin "1")
-    (pin "2")
-    (pin "3")
-    (pin "4")
-    (instances
-      (project "stm32"
-        (path "/cc56704c-71b4-401e-bec6-203f83946289/10666af3-dfc7-46de-8942-14bdd4d81ac1"
-          (reference "J7") (unit 1)
-        )
-        (path "/cc56704c-71b4-401e-bec6-203f83946289/373d422b-50db-40b1-b72f-ec977be46bcc"
-          (reference "J15") (unit 1)
-        )
-      )
-    )
-  )
 )
